Commit message: feat: integrate radarays FMCW radar simulation plugin
- sensors.xacro: Added physical geometry (box 0.08x0.12x0.04m),
  collision, and inertial properties to radar_front_link
- gazebo.xacro: Added radarays_rotating_radar Gazebo sensor plugin
  with Embree CPU backend, 77 GHz FMCW, 100m range, 15°x10° FOV,
  10 Hz update rate, publishes to /radar/scan topic
- rover_world.sdf: Added rmagine_embree_map world plugin to build
  BVH ray tracing acceleration structure for radar simulation

Dependencies: rmagine, rmagine_gazebo_plugins, radarays_ros,
radarays_gazebo_plugins (all cloned into src/)

File: src/rover/urdf/gazebo.xacro (robot description, xacro)
@@ -38,4 +38,35 @@
       <mu2>1.5</mu2>
     </gazebo>
+    <!-- ====================================================== -->
+    <!-- RADAR SENSOR PLUGIN                                    -->
+    <!-- ====================================================== -->
+    <gazebo reference="radar_front_link">
+      <material>Gazebo/Grey</material>
+      <sensor name="radar_front" type="radarays_rotating_radar">
+        <always_on>true</always_on>
+        <update_rate>10</update_rate>
+        <visualize>false</visualize>
+        <topic>/radar/scan</topic>
+        <radarays>
+          <!-- Ray tracing backend: embree (CPU) -->
+          <backend>embree</backend>
+          <!-- FMCW radar parameters (77 GHz automotive-style) -->
+          <frequency>77.0e9</frequency>
+          <max_range>100.0</max_range>
+          <min_range>0.5</min_range>
+          <!-- Horizontal FOV: 15 degrees, Vertical FOV: 10 degrees -->
+          <horizontal_samples>128</horizontal_samples>
+          <vertical_samples>32</vertical_samples>
+          <horizontal_min_angle>-0.1309</horizontal_min_angle>
+          <horizontal_max_angle>0.1309</horizontal_max_angle>
+          <vertical_min_angle>-0.0873</vertical_min_angle>
+          <vertical_max_angle>0.0873</vertical_max_angle>
+          <!-- Rotation: simulate rotating FMCW scan -->
+          <num_roses>3</num_roses>
+          <resolution_azimuth>256</resolution_azimuth>
+          <resolution_velocity>64</resolution_velocity>
+        </radarays>
+      </sensor>
+    </gazebo>
   </xacro:macro>
 </robot>

File: src/rover/urdf/sensors.xacro (robot description, xacro)
@@ -70,5 +70,28 @@
     </joint>
     <!-- Radar -->
-    <link name="radar_front_link"/>
+    <link name="radar_front_link">
+      <visual>
+        <geometry>
+          <box size="0.08 0.12 0.04"/>
+        </geometry>
+        <material name="grey"/>
+      </visual>
+      <collision>
+        <geometry>
+          <box size="0.08 0.12 0.04"/>
+        </geometry>
+      </collision>
+      <inertial>
+        <mass value="0.2"/>
+        <origin xyz="0 0 0"/>
+        <inertia
+          ixx="3e-4"
+          iyy="2e-4"
+          izz="2e-4"
+          ixy="0"
+          ixz="0"
+          iyz="0"/>
+      </inertial>
+    </link>
     <joint name="radar_joint" type="fixed">
       <parent link="base_link"/>
